File: Circuito - Kicad/Circuito - Kicad.kicad_sch (KiCad schematic)
At the start: 11 parts, among them U1 4N25, U2 MOC3021M

Commit message: KiCad Circuit Improvement
Other:
- note added: "Circuito de Funcionamiento"
- note added: "Circuito de Lectura"
- note added: "Circuito diseñado y simulado en Proteus"
- moved on the sheet: AC, Calentador, R1, R2, R3, R4, SH1, Sensor, Triac, U1, U2

Commit message: KiCad Improvement | Again
Parts:
- renumbered AC to AC1, Calentador to Calentador1, Sensor to Sensor1, Triac to Triac1
Changed lines of the file:
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@@
 		(dnp no)
 		(fields_autoplaced yes)
-		(property "Reference" "AC"
+		(property "Reference" "AC1"
 			(at 73.152 170.1799 0)
 			(effects
@@
 			(project "Circuito - Kicad"
 				(path "/5c956fab-8f3e-46bb-9b36-ad0edafc8e4e"
-					(reference "AC")
+					(reference "AC1")
 					(unit 1)
 				)
@@
 		(dnp no)
 		(fields_autoplaced yes)
-		(property "Reference" "Sensor"
+		(property "Reference" "Sensor1"
 			(at 30.988 136.652 0)
 			(effects
@@
 			(project ""
 				(path "/5c956fab-8f3e-46bb-9b36-ad0edafc8e4e"
-					(reference "Sensor")
+					(reference "Sensor1")
 					(unit 1)
 				)
@@
 		(on_board yes)
 		(dnp no)
-		(property "Reference" "Triac"
+		(property "Reference" "Triac1"
 			(at 242.57 92.71 0)
 			(effects
@@
 			(project ""
 				(path "/5c956fab-8f3e-46bb-9b36-ad0edafc8e4e"
-					(reference "Triac")
+					(reference "Triac1")
 					(unit 1)
 				)
@@
 		(on_board yes)
 		(dnp no)
-		(property "Reference" "Calentador"
+		(property "Reference" "Calentador1"
 			(at 255.27 68.8339 90)
 			(effects
@@
 			(project ""
 				(path "/5c956fab-8f3e-46bb-9b36-ad0edafc8e4e"
-					(reference "Calentador")
-					(unit 1)
-				)
+					(reference "Calentador1")
+					(unit 1)
+				)

Commit message: Kicad | PCB Improvement
Parts:
- R1, R2, R3, R4: footprint (none) -> Resistor_THT:R_Axial_DIN0207_L6.3mm_D2.5mm_P10.16mm_Horizontal
- U2: footprint (none) -> MOC3021:DIP762W45P254L889H508Q6
- renumbered AC1 to Alterna1
Changed lines of the file:
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@@
 			)
 		)
-		(property "Footprint" ""
+		(property "Footprint" "Resistor_THT:R_Axial_DIN0207_L6.3mm_D2.5mm_P10.16mm_Horizontal"
 			(at 190.5 88.646 90)
 			(effects
@@
 			)
 		)
-		(property "Footprint" ""
+		(property "Footprint" "Resistor_THT:R_Axial_DIN0207_L6.3mm_D2.5mm_P10.16mm_Horizontal"
 			(at 121.158 42.926 90)
 			(effects
@@
 		(dnp no)
 		(fields_autoplaced yes)
-		(property "Reference" "AC1"
-			(at 73.152 170.1799 0)
+		(property "Reference" "Alterna1"
+			(at 72.39 170.1799 0)
 			(effects
 				(font
@@
 		)
 		(property "Value" "TB_1X2"
-			(at 73.152 172.7199 0)
+			(at 72.39 172.7199 0)
 			(effects
 				(font
@@
 			(project "Circuito - Kicad"
 				(path "/5c956fab-8f3e-46bb-9b36-ad0edafc8e4e"
-					(reference "AC1")
+					(reference "Alterna1")
 					(unit 1)
 				)
@@
 			)
 		)
-		(property "Footprint" ""
+		(property "Footprint" "MOC3021:DIP762W45P254L889H508Q6"
 			(at 203.2 98.044 0)
 			(effects
@@
 			)
 		)
-		(property "Footprint" ""
+		(property "Footprint" "Resistor_THT:R_Axial_DIN0207_L6.3mm_D2.5mm_P10.16mm_Horizontal"
 			(at 229.87 78.486 90)
 			(effects
@@
 			)
 		)
-		(property "Footprint" ""
+		(property "Footprint" "Resistor_THT:R_Axial_DIN0207_L6.3mm_D2.5mm_P10.16mm_Horizontal"
 			(at 156.718 29.21 90)
 			(effects

Commit message: Kicad | PCB Added
Parts:
- Triac1: footprint (none) -> BT136:TO220AB
Changed lines of the file:
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@@
 			)
 		)
-		(property "Footprint" ""
+		(property "Footprint" "BT136:TO220AB"
 			(at 240.665 92.329 90)
 			(effects

Commit message: PCB Improvement
Parts:
- Triac1: footprint BT136:TO220AB -> BT139-600E:TO255P1040X460X1975-3
Changed lines of the file:
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@@
 			)
 		)
-		(property "Footprint" "BT136:TO220AB"
+		(property "Footprint" "BT139-600E:TO255P1040X460X1975-3"
 			(at 240.665 92.329 90)
 			(effects

Commit message: Kicad Improvement
Parts:
- removed Sensor1: TB_1X3, EESTN5:BORNERA3, symbol EESTN5e:TB_1X3
- added Potenciometro1: TB_1X3, EESTN5:BORNERA3, symbol EESTN5:TB_1X3
Connections:
- net +5V is gone; now on net VCC: U1.5
- net GND: now also SH1.GND1 (GND/1), Potenciometro1.3
- net PIN_A0: now also Potenciometro1.2
- net VCC: now reaches SH1.5V
- net VCC: now also Potenciometro1.1
Changed lines of the file:
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@@
 	(wire
 		(pts
-			(xy 38.608 149.352) (xy 56.388 149.352)
+			(xy 37.846 144.272) (xy 48.26 144.272)
 		)
 		(stroke
@@
 	(wire
 		(pts
-			(xy 28.194 169.672) (xy 28.194 176.022)
+			(xy 37.846 154.432) (xy 49.022 154.432)
 		)
 		(stroke
@@
 	(wire
 		(pts
+			(xy 24.4094 58.674) (xy 33.528 58.674)
+		)
+		(stroke
+			(width 0)
+			(type default)
+		)
+	)
+	(wire
+		(pts
 			(xy 72.898 64.389) (xy 80.772 64.389)
 		)
@@
 	(wire
 		(pts
+			(xy 26.416 55.499) (xy 26.416 40.894)
+		)
+		(stroke
+			(width 0)
+			(type default)
+		)
+	)
+	(wire
+		(pts
 			(xy 238.76 101.6) (xy 262.382 101.6)
 		)
@@
 		)
 	)
+	(wire
+		(pts
+			(xy 26.416 55.499) (xy 33.528 55.499)
+		)
+		(stroke
+			(width 0)
+			(type default)
+		)
+	)
+	(wire
+		(pts
+			(xy 24.4094 45.466) (xy 24.4094 58.674)
+		)
+		(stroke
+			(width 0)
+			(type default)
+		)
+	)
 	(polyline
 		(pts
@@
 	(wire
 		(pts
+			(xy 37.846 149.352) (xy 66.04 149.352)
+		)
+		(stroke
+			(width 0)
+			(type default)
+		)
+	)
+	(wire
+		(pts
 			(xy 246.38 77.724) (xy 246.38 80.264)
 		)
@@
 	(wire
 		(pts
-			(xy 35.814 169.672) (xy 35.814 176.022)
+			(xy 24.4094 45.466) (xy 19.558 45.466)
 		)
 		(stroke
@@
 	)
 	(image
-		(at -105.664 68.6816)
+		(at -96.774 68.9356)
 		(data "/9j/4AAQSkZJRgABAQEAYABgAAD/2wBDAAMCAgICAgMCAgIDAwMDBAYEBAQEBAgGBgUGCQgKCgkI"
 			"CQkKDA8MCgsOCwkJDRENDg8QEBEQCgwSExIQEw8QEBD/2wBDAQMDAwQDBAgEBAgQCwkLEBAQEBAQ"
@@
 	(global_label "GND"
 		(shape input)
-		(at 38.608 154.432 0)
+		(at 49.022 154.432 0)
 		(fields_autoplaced yes)
 		(effects
@@
 		)
 		(property "Intersheetrefs" "${INTERSHEET_REFS}"
-			(at 45.4637 154.432 0)
+			(at 55.8777 154.432 0)
 			(effects
 				(font
@@
 	(global_label "VCC"
 		(shape input)
-		(at 28.194 176.022 270)
+		(at 26.416 40.894 180)
 		(fields_autoplaced yes)
 		(effects
@@
 		)
 		(property "Intersheetrefs" ""
-			(at 28.194 182.6358 90)
+			(at 19.8022 40.894 0)
 			(effects
 				(font
@@
 	(global_label "VCC"
 		(shape input)
-		(at 38.608 144.272 0)
+		(at 48.26 144.272 0)
 		(fields_autoplaced yes)
 		(effects
@@
 		)
 		(property "Intersheetrefs" ""
-			(at 45.2218 144.272 0)
+			(at 54.8738 144.272 0)
 			(effects
 				(font
@@
 	(global_label "GND"
 		(shape input)
-		(at 35.814 176.022 270)
+		(at 19.558 45.466 180)
 		(fields_autoplaced yes)
 		(effects
@@
 		)
 		(property "Intersheetrefs" "${INTERSHEET_REFS}"
-			(at 35.814 182.8777 90)
+			(at 12.7023 45.466 0)
 			(effects
 				(font
@@
 	(global_label "PIN_A0"
 		(shape input)
-		(at 56.388 149.352 0)
+		(at 66.04 149.352 0)
 		(fields_autoplaced yes)
 		(effects
@@
 		)
 		(property "Intersheetrefs" "${INTERSHEET_REFS}"
-			(at 65.8442 149.352 0)
+			(at 75.4962 149.352 0)
 			(effects
 				(font
@@
 	)
 	(symbol
+		(lib_id "EESTN5:TB_1X3")
+		(at 28.956 146.812 0)
+		(unit 1)
+		(exclude_from_sim no)
+		(in_bom yes)
+		(on_board yes)
+		(dnp no)
+		(fields_autoplaced yes)
+		(property "Reference" "Potenciometro1"
+			(at 30.226 137.16 0)
+			(effects
+				(font
+					(size 1.524 1.524)
+				)
+			)
+		)
+		(property "Value" "TB_1X3"
+			(at 30.226 139.7 0)
+			(effects
+				(font
+					(size 1.524 1.524)
+				)
+			)
+		)
+		(property "Footprint" "EESTN5:BORNERA3"
+			(at 27.686 145.542 0)
+			(effects
+				(font
+					(size 1.524 1.524)
+				)
+				(hide yes)
+			)
+		)
+		(property "Datasheet" ""
+			(at 27.686 145.542 0)
+			(effects
+				(font
+					(size 1.524 1.524)
+				)
+			)
+		)
+		(property "Description" ""
+			(at 28.956 146.812 0)
+			(effects
+				(font
+					(size 1.27 1.27)
+				)
+				(hide yes)
+			)
+		)
+		(pin "2"
+		)
+		(pin "1"
+		)
+		(pin "3"
+		)
+		(instances
+			(project ""
+				(path "/5c956fab-8f3e-46bb-9b36-ad0edafc8e4e"
+					(reference "Potenciometro1")
+					(unit 1)
+				)
+			)
+		)
+	)
+	(symbol
 		(lib_id "Device:R")
 		(at 190.5 90.424 270)
@@
 	)
 	(symbol
-		(lib_id "power:+5V")
-		(at 28.194 169.672 0)
-		(unit 1)
-		(exclude_from_sim no)
-		(in_bom yes)
-		(on_board yes)
-		(dnp no)
-		(fields_autoplaced yes)
-		(property "Reference" "#PWR01"
-			(at 28.194 173.482 0)
-			(effects
-				(font
-					(size 1.27 1.27)
-				)
-				(hide yes)
-			)
-		)
-		(property "Value" "+5V"
-			(at 28.194 164.592 0)
-			(effects
-				(font
-					(size 1.27 1.27)
-				)
-			)
-		)
-		(property "Footprint" ""
-			(at 28.194 169.672 0)
-			(effects
-				(font
-					(size 1.27 1.27)
-				)
-				(hide yes)
-			)
-		)
-		(property "Datasheet" ""
-			(at 28.194 169.672 0)
-			(effects
-				(font
-					(size 1.27 1.27)
-				)
-				(hide yes)
-			)
-		)
-		(property "Description" "Power symbol creates a global label with name \"+5V\""
-			(at 28.194 169.672 0)
-			(effects
-				(font
-					(size 1.27 1.27)
-				)
-				(hide yes)
-			)
-		)
-		(pin "1"
-		)
-		(instances
-			(project ""
-				(path "/5c956fab-8f3e-46bb-9b36-ad0edafc8e4e"
-					(reference "#PWR01")
-					(unit 1)
-				)
-			)
-		)
-	)
-	(symbol
-		(lib_id "EESTN5e:TB_1X3")
-		(at 29.718 146.812 0)
-		(unit 1)
-		(exclude_from_sim no)
-		(in_bom yes)
-		(on_board yes)
-		(dnp no)
-		(fields_autoplaced yes)
-		(property "Reference" "Sensor1"
-			(at 30.988 136.652 0)
-			(effects
-				(font
-					(size 1.524 1.524)
-				)
-			)
-		)
-		(property "Value" "TB_1X3"
-			(at 30.988 139.192 0)
-			(effects
-				(font
-					(size 1.524 1.524)
-				)
-			)
-		)
-		(property "Footprint" "EESTN5:BORNERA3"
-			(at 28.448 145.542 0)
-			(effects
-				(font
-					(size 1.524 1.524)
-				)
-				(hide yes)
-			)
-		)
-		(property "Datasheet" ""
-			(at 28.448 145.542 0)
-			(effects
-				(font
-					(size 1.524 1.524)
-				)
-			)
-		)
-		(property "Description" ""
-			(at 29.718 146.812 0)
-			(effects
-				(font
-					(size 1.27 1.27)
-				)
-				(hide yes)
-			)
-		)
-		(pin "2"
-		)
-		(pin "3"
-		)
-		(pin "1"
-		)
-		(instances
-			(project ""
-				(path "/5c956fab-8f3e-46bb-9b36-ad0edafc8e4e"
-					(reference "Sensor1")
-					(unit 1)
-				)
-			)
-		)
-	)
-	(symbol
 		(lib_id "Triac_Thyristor:Generic_Triac_A1A2G")
 		(at 238.76 92.964 0)
@@
 					(unit 1)
 				)
-			)
-		)
-	)
-	(symbol
-		(lib_id "power:GND")
-		(at 35.814 169.672 180)
-		(unit 1)
-		(exclude_from_sim no)
-		(in_bom yes)
-		(on_board yes)
-		(dnp no)
-		(fields_autoplaced yes)
-		(property "Reference" "#PWR02"
-			(at 35.814 163.322 0)
-			(effects
-				(font
-					(size 1.27 1.27)
-				)
-				(hide yes)
-			)
-		)
-		(property "Value" "GND"
-			(at 35.814 164.592 0)
-			(effects
-				(font
-					(size 1.27 1.27)
-				)
-			)
-		)
-		(property "Footprint" ""
-			(at 35.814 169.672 0)
-			(effects
-				(font
-					(size 1.27 1.27)
-				)
-				(hide yes)
-			)
-		)
-		(property "Datasheet" ""
-			(at 35.814 169.672 0)
-			(effects
-				(font
-					(size 1.27 1.27)
-				)
-				(hide yes)
-			)
-		)
-		(property "Description" "Power symbol creates a global label with name \"GND\" , ground"
-			(at 35.814 169.672 0)
-			(effects
-				(font
-					(size 1.27 1.27)
-				)
-				(hide yes)
-			)
-		)
-		(pin "1"
-		)
-		(instances
-			(project ""
-				(path "/5c956fab-8f3e-46bb-9b36-ad0edafc8e4e"
-					(reference "#PWR02")
-					(unit 1)
-				)

Commit message: Kicad | Schematic Improvement
Parts:
- removed Potenciometro1: TB_1X3, EESTN5:BORNERA3, symbol EESTN5:TB_1X3
- removed SH1: ARDUINO_as_UNO, EESTN5:ARDUINO_UNO_R2_CONTOUR, symbol EESTN5e:ARDUINO_as_UNO
- added Alimentación1: Alimentación | Arduino, EESTN5:Pin_Header_2, symbol Connector:Conn_01x02_Pin
- added Datos1: Datos, EESTN5:Pin_Header_3, symbol Connector:Conn_01x03_Pin
- Alterna1: value TB_1X2 -> Alterna
- Calentador1: value TB_1X2 -> Calentador
- Triac1: value Generic_Triac_A1A2G -> Triac
Connections:
- net GND: now also Alimentación1.2 (Pin_2)
- net PIN_2: now also R4.1, U1.4, Datos1.1 (Pin_1)
- net PIN_7: now also Datos1.2 (Pin_2)
- net PIN_A0: now also Datos1.3 (Pin_3)
- net VCC: now also Alimentación1.1 (Pin_1)
Other:
- note removed: "Control | Sensor"
- moved on the sheet: Alterna1, R4
