File: Circuito - Kicad/dimmer.kicad_pcb (KiCad board)
At the start: 2 copper layers, 74 parts, among them J1 DCJ200-10-A-XX-K_REVA, J2 DHT11, T1592 Datos, U1 MOC3021M, U2 4N25, U4 5V, U5 MOC3021M

Commit message: Code Improvement [C++] | Pretty Code
Parts:
- removed the 4.7K1 at (68.5, 72.7)
- removed the 5K1 at (97.0, 72.0)
- removed the A1 at (74.2, 41.7)
- removed the Alterna1 at (83.2, 120.7)
- removed the C1 at (127.5, 83.7)
- removed the C2 at (111.0, 50.2)
- removed the C3 at (118.0, 46.7)
- removed the C4 at (67.2, 83.5)
- removed the Calentador1 at (108.7, 120.7)
- removed the Calentador2 at (56.2, 120.7)
- removed the D1 at (111.7, 59.2)
- removed the DS18B20 at (64.2, 71.7)
- removed the G*** at (51.6, 46.6) (x2)
- removed the J1 at (124.2, 36.7)
- removed the J2 at (101.5, 65.2)
- removed the R1 at (112.7, 85.7)
- removed the R10 at (52.7, 103.7)
- removed the R11 at (58.2, 103.7)
- removed the R12 at (60.5, 98.8)
- removed the R2 at (112.2, 103.7)
- removed the R3 at (106.2, 103.7)
- removed the R4 at (91.0, 87.7)
- removed the R5 at (78.6, 105.7)
- removed the R6 at (55.0, 87.9)
- removed the R600 at (118.7, 99.1)
- removed the R7 at (111.7, 56.0)
- removed the R8 at (101.5, 55.2)
- removed the R9 at (101.5, 51.8)
- removed the T1592 at (107.5, 70.0)
- removed the Triac1 at (109.2, 111.7)
- removed the Triac2 at (56.2, 112.7)
- removed the U1 at (110.2, 94.7)
- removed the U2 at (78.1, 97.7)
- removed the U4 at (117.0, 52.7)
- removed the U5 at (52.5, 95.2)
- removed the YF-S201 at (95.5, 43.7)
Routing:
- net Vivo: track 346.5 -> 173.2 mm
- net 5V: track 206.0 -> 103.0 mm
- net 3.3V: track 172.0 -> 86.0 mm
- net Neutro: track 164.5 -> 82.2 mm
- net D3: track 137.8 -> 68.9 mm
- net D6: track 106.8 -> 53.4 mm
- net D2: track 101.2 -> 50.6 mm
- net D5: track 88.2 -> 44.1 mm
- net D4: track 84.9 -> 42.4 mm
- net Net-(Triac1-A2): track 62.5 -> 31.3 mm
- net Net-(Triac2-A2): track 53.3 -> 26.6 mm
- net A1: track 48.2 -> 24.1 mm
- net VIN: track 45.7 -> 22.9 mm
- net A0: track 39.5 -> 19.8 mm
- net D7: track 33.9 -> 16.9 mm
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